Commit message: Adding chemical partical sensor for plume simulation

File: uuv_descriptions/urdf/rexrov_sensors.xacro (robot description, xacro)
@@ -54,3 +54,10 @@
     parent_link="${namespace}/base_link"
     inertial_reference_frame="${inertial_reference_frame}" />
+  <!-- Mount chemical particle concentration sensor -->
+  <xacro:default_chemical_concentration_sensor_macro
+    namespace="${namespace}"
+    parent_link="${namespace}/base_link"
+    inertial_reference_frame="${inertial_reference_frame}">
+    <origin xyz="0 0 0" rpy="0 0 0"/>
+  </xacro:default_chemical_concentration_sensor_macro>
 </robot>
